File: PCB/Guys-split-keyboard/Guys-split-keyboard.kicad_sch (KiCad schematic)
At the start: 0 parts

Commit message: work
Other:
- added sheet left (half.kicad_sch)
- added sheet right (half.kicad_sch)
Changed lines of the file:
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@@
 	(generator_version "9.0")
 	(paper "A4")
+	(sheet
+		(at 160.02 72.39)
+		(size 104.14 73.66)
+		(exclude_from_sim no)
+		(in_bom yes)
+		(on_board yes)
+		(dnp no)
+		(fields_autoplaced yes)
+		(stroke
+			(width 0.1524)
+			(type solid)
+		)
+		(fill
+			(color 0 0 0 0.0000)
+		)
+		(property "Sheetname" "right"
+			(at 160.02 71.6784 0)
+			(effects
+				(font
+					(size 1.27 1.27)
+				)
+				(justify left bottom)
+			)
+		)
+		(property "Sheetfile" "half.kicad_sch"
+			(at 160.02 146.6346 0)
+			(effects
+				(font
+					(size 1.27 1.27)
+				)
+				(justify left top)
+			)
+		)
+		(instances
+			(project "Guys-split-keyboard"
+				(path "/89922203-b126-4628-8264-14224bcab0ba"
+					(page "3")
+				)
+			)
+		)
+	)
+	(sheet
+		(at 45.72 72.39)
+		(size 97.79 73.66)
+		(exclude_from_sim no)
+		(in_bom yes)
+		(on_board yes)
+		(dnp no)
+		(fields_autoplaced yes)
+		(stroke
+			(width 0.1524)
+			(type solid)
+		)
+		(fill
+			(color 0 0 0 0.0000)
+		)
+		(property "Sheetname" "left"
+			(at 45.72 71.6784 0)
+			(effects
+				(font
+					(size 1.27 1.27)
+				)
+				(justify left bottom)
+			)
+		)
+		(property "Sheetfile" "half.kicad_sch"
+			(at 45.72 146.6346 0)
+			(effects
+				(font
+					(size 1.27 1.27)
+				)
+				(justify left top)
+			)
+		)
+		(instances
+			(project "Guys-split-keyboard"
+				(path "/89922203-b126-4628-8264-14224bcab0ba"
+					(page "2")
+				)
+			)
+		)
+	)
 	(sheet_instances
 		(path "/"
