File: PCB/Guys-split-keyboard/_autosave-half.kicad_sch (KiCad schematic)
At the start: 51 parts, among them SW1 SW_Push, SW11 SW_Push, SW13 SW_Push, SW14 SW_Push, SW15 SW_Push, SW16 SW_Push, SW17 SW_Push, SW18 SW_Push, SW25 SW_Push, SW26 SW_Push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

Commit message: some more work
Parts:
- U1: footprint wirelesskeyboard:modified-XIAO-nRF52840-SMD -> Moddedxiao:modified-XIAO-nRF52840-SMD
Changed lines of the file:
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@@
 			)
 		)
-		(property "Footprint" "wirelesskeyboard:modified-XIAO-nRF52840-SMD"
+		(property "Footprint" "Moddedxiao:modified-XIAO-nRF52840-SMD"
 			(at 50.8 57.15 0)
 			(effects
