File: PCB V2/Guys-split-keyboard/Guys-split-keyboard.kicad_pcb (KiCad board)
At the start: 2 copper layers, 161 x 98 mm, 55 parts, among them SW1 SW_Push, SW10 SW_Push, SW11 SW_Push, SW12 SW_Push, SW13 SW_Push, SW14 SW_Push, SW15 SW_Push, SW16 SW_Push, SW17 SW_Push, SW18 SW_Push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

Commit message: pcb V1 and V2
Parts:
- moved D17 60.4 mm to (250.6, 93.6)
- moved D18 60.4 mm to (269.6, 93.6)
- moved D16 58.2 mm to (174.4, 91.2)
- moved D14 55.7 mm to (193.4, 88.8)
- moved D15 55.7 mm to (231.6, 88.8)
- moved D13 53.3 mm to (212.6, 86.4)
- moved D11 42.3 mm to (250.6, 74.6)
- moved D12 42.2 mm to (269.6, 74.6)
- moved D10 40.4 mm to (174.4, 72.1)
- moved H5 39.9 mm to (159.0, 40.0)
- moved D8 38.0 mm to (193.4, 69.8)
- moved D9 37.7 mm to (231.6, 69.8)
- moved D7 35.4 mm to (212.4, 67.3)
- moved D5 27.0 mm to (250.6, 55.6)
- moved D6 26.7 mm to (269.6, 55.6)
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Routing:
- net Net-(D18-A): track 64.6 -> 7.66 mm
- net Net-(D17-A): track 64.3 -> 7.67 mm
- net Net-(D16-A): track 60.9 -> 7.67 mm
- net Net-(D15-A): track 59.3 -> 7.73 mm
- net Net-(D14-A): track 58.8 -> 7.63 mm
- net Net-(D13-A): track 56.6 -> 7.79 mm
- net Row2: track 179.9 -> 138.2 mm
- net Net-(D11-A): track 45.1 -> 7.65 mm
- net Net-(D12-A): track 45.0 -> 7.64 mm
- net Net-(D10-A): track 43.7 -> 7.69 mm
- net Net-(D8-A): track 41.0 -> 7.61 mm
- net Net-(D9-A): track 40.6 -> 7.71 mm
- net Net-(D7-A): track 38.4 -> 7.61 mm
- net Row3: track 130.2 -> 158.7 mm
- net Net-(D6-A): track 28.0 -> 7.61 mm
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Other:
- board size 161 x 98 mm -> 162 x 94 mm
- board text added: "D4"
