File: PCB V2/Guys-split-keyboard/half.kicad_sch (KiCad schematic)
At the start: 51 parts, among them SW1 SW_Push, SW11 SW_Push, SW13 SW_Push, SW14 SW_Push, SW15 SW_Push, SW16 SW_Push, SW17 SW_Push, SW18 SW_Push, SW25 SW_Push, SW26 SW_Push, SW27 SW_Push, SW28 SW_Push, SW29 SW_Push, SW3 SW_Push, SW30 SW_Push, SW37 SW_Push, SW38 SW_Push, SW39 SW_Push, SW5 SW_Push, SW7 SW_Push, SW9 SW_Push, U1 XIAO-nRF52840-SMD

Commit message: pcb V1 and V2
Parts:
- added H5, H6, H7, H8: MountingHole, TestPoint:TestPoint_Loop_D3.80mm_Drill2.8mm, symbol Mechanical:MountingHole
- D1: footprint Diode_SMD:D_SOD-123 -> Diode_THT:D_DO-35_SOD27_P7.62mm_Horizontal
- D10: renamed from D16; footprint Diode_SMD:D_SOD-123 -> Diode_THT:D_DO-35_SOD27_P7.62mm_Horizontal
- D11: renamed from D17; footprint Diode_SMD:D_SOD-123 -> Diode_THT:D_DO-35_SOD27_P7.62mm_Horizontal
- D12: renamed from D18; footprint Diode_SMD:D_SOD-123 -> Diode_THT:D_DO-35_SOD27_P7.62mm_Horizontal
- D13: renamed from D25; footprint Diode_SMD:D_SOD-123 -> Diode_THT:D_DO-35_SOD27_P7.62mm_Horizontal
- D14: renamed from D26; footprint Diode_SMD:D_SOD-123 -> Diode_THT:D_DO-35_SOD27_P7.62mm_Horizontal
- D15: renamed from D27; footprint Diode_SMD:D_SOD-123 -> Diode_THT:D_DO-35_SOD27_P7.62mm_Horizontal
- D16: renamed from D28; footprint Diode_SMD:D_SOD-123 -> Diode_THT:D_DO-35_SOD27_P7.62mm_Horizontal
- D17: renamed from D29; footprint Diode_SMD:D_SOD-123 -> Diode_THT:D_DO-35_SOD27_P7.62mm_Horizontal
- D18: renamed from D30; footprint Diode_SMD:D_SOD-123 -> Diode_THT:D_DO-35_SOD27_P7.62mm_Horizontal
- D19: renamed from D37; footprint Diode_SMD:D_SOD-123 -> Diode_THT:D_DO-35_SOD27_P7.62mm_Horizontal
- D2: renamed from D3; footprint Diode_SMD:D_SOD-123 -> Diode_THT:D_DO-35_SOD27_P7.62mm_Horizontal
- D20: renamed from D38; footprint Diode_SMD:D_SOD-123 -> Diode_THT:D_DO-35_SOD27_P7.62mm_Horizontal
- D21: renamed from D39; footprint Diode_SMD:D_SOD-123 -> Diode_THT:D_DO-35_SOD27_P7.62mm_Horizontal
- D3: renamed from D5; footprint Diode_SMD:D_SOD-123 -> Diode_THT:D_DO-35_SOD27_P7.62mm_Horizontal
- D4: renamed from D7; footprint Diode_SMD:D_SOD-123 -> Diode_THT:D_DO-35_SOD27_P7.62mm_Horizontal
- D5: renamed from D9; footprint Diode_SMD:D_SOD-123 -> Diode_THT:D_DO-35_SOD27_P7.62mm_Horizontal
- D6: renamed from D11; footprint Diode_SMD:D_SOD-123 -> Diode_THT:D_DO-35_SOD27_P7.62mm_Horizontal
- D7: renamed from D13; footprint Diode_SMD:D_SOD-123 -> Diode_THT:D_DO-35_SOD27_P7.62mm_Horizontal
- D8: renamed from D14; footprint Diode_SMD:D_SOD-123 -> Diode_THT:D_DO-35_SOD27_P7.62mm_Horizontal
- D9: renamed from D15; footprint Diode_SMD:D_SOD-123 -> Diode_THT:D_DO-35_SOD27_P7.62mm_Horizontal
- R1: footprint Resistor_SMD:R_0805_2012Metric -> Resistor_THT:R_Axial_DIN0207_L6.3mm_D2.5mm_P7.62mm_Horizontal
- R2: renamed from R3; footprint Resistor_SMD:R_0805_2012Metric -> Resistor_THT:R_Axial_DIN0207_L6.3mm_D2.5mm_P7.62mm_Horizontal
- SW20: renamed from SW38; footprint GateronKS33Solder:Gateron-KS33-Solderable-1U -> GateronKS33Solder:Gateron-KS33-Solderable-2U
- renumbered H3 to H2, H5 to H3, H7 to H4, SW16 to SW10, SW17 to SW11, SW18 to SW12, SW25 to SW13, SW26 to SW14, SW27 to SW15, SW28 to SW16, SW29 to SW17, SW30 to SW18, SW37 to SW19, SW3 to SW2, SW39 to SW21, SW5 to SW3, SW7 to SW4, SW9 to SW5, SW11 to SW6, SW13 to SW7, SW14 to SW8, SW15 to SW9, TP3 to TP2
Other:
- note added: "mounting holes"
- note added: "mousbites"

Commit message: I forgot the other half, todo later
Parts:
- renumbered D9 to D10, D15 to D11, D21 to D12, D4 to D13, D10 to D14, D16 to D15, D5 to D16, D11 to D17, D17 to D18, D6 to D19, D7 to D2, D12 to D20, D18 to D21, D13 to D3, D19 to D4, D2 to D5, D8 to D6, D14 to D7, D20 to D8, D3 to D9, H5 to H2, H2 to H3, H6 to H4, H3 to H5, H7 to H6, H4 to H7, SW9 to SW10, SW15 to SW11, SW21 to SW12, SW4 to SW13, SW10 to SW14, SW16 to SW15, SW5 to SW16, SW11 to SW17, SW17 to SW18, SW6 to SW19, SW7 to SW2, SW12 to SW20, SW18 to SW21, SW13 to SW3, SW19 to SW4, SW2 to SW5, SW8 to SW6, SW14 to SW7, SW20 to SW8, SW3 to SW9
Connections:
- net BTPin renamed BTPin2
- net Col1 renamed Col11
- net Col2 renamed Col22
- net Col3 renamed Col33
- net Col4 renamed Col44
- net Col5 renamed Col55
- net Col6 renamed Col66
- net GND renamed GND2
- net GND2: no longer U1.13 (GND)
- net Row1 renamed Row11
- net Row2 renamed Row22
- net Row3 renamed Row33
- net Row4 renamed Row44
- net VBAT renamed VBAT2
- net VBAT2: now also U1.13 (GND)
