File: PCB V2/Guys-split-keyboard/Guys-split-keyboardV2.kicad_pcb (KiCad board)
At the start: 2 copper layers, 162 x 94 mm, 55 parts, among them SW1 SW_Push, SW10 SW_Push, SW11 SW_Push, SW12 SW_Push, SW13 SW_Push, SW14 SW_Push, SW15 SW_Push, SW16 SW_Push, SW17 SW_Push, SW18 SW_Push, SW19 SW_Push, SW2 SW_Push, SW20 SW_Push, SW21 SW_Push, SW3 SW_Push, SW4 SW_Push, SW5 SW_Push, SW6 SW_Push, SW7 SW_Push, SW8 SW_Push, SW9 SW_Push, U1 XIAO-nRF52840-SMD

Commit message: I forgot the other half, todo later
Parts:
- moved D19 92.1 mm to (178.7, 40.8)
- moved D20 92.1 mm to (178.7, 59.8)
- moved D21 92.1 mm to (178.7, 78.8)
- moved D10 92.1 mm to (140.7, 55.0)
- moved D11 92.1 mm to (140.7, 74.0)
- moved D12 92.1 mm to (75.1, 99.7)
- moved D13 92.1 mm to (83.5, 38.2)
- moved D14 92.1 mm to (83.5, 57.3)
- moved D15 92.1 mm to (83.5, 76.4)
- moved D16 92.1 mm to (159.7, 40.8)
- moved D17 92.1 mm to (159.7, 59.8)
- moved D18 92.1 mm to (159.7, 78.8)
- moved D2 92.1 mm to (121.5, 52.5)
- moved D5 92.1 mm to (102.5, 36.0)
- moved D6 92.1 mm to (102.5, 55.0)
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- renumbered D9 to D10, D15 to D11, D21 to D12, D4 to D13, D10 to D14, D16 to D15, D5 to D16, D11 to D17, D17 to D18, D6 to D19, D7 to D2, D12 to D20, D18 to D21, D13 to D3, D19 to D4, D2 to D5, D8 to D6, D14 to D7, D20 to D8, D3 to D9, H5 to H2, H2 to H3, H6 to H4, H3 to H5, H7 to H6, H4 to H7, SW9 to SW10, SW15 to SW11, SW21 to SW12, SW4 to SW13, SW10 to SW14, SW16 to SW15, SW5 to SW16, SW11 to SW17, SW17 to SW18, SW6 to SW19, SW7 to SW2, SW12 to SW20, SW18 to SW21, SW13 to SW3, SW19 to SW4, SW2 to SW5, SW8 to SW6, SW14 to SW7, SW20 to SW8, SW3 to SW9
Other:
- board text added: "Guy's Split Keyboard"
- board text added: "right side"

Commit message: added other half
Parts:
- added D1: D, Diode_THT:D_DO-35_SOD27_P7.62mm_Horizontal, F.Cu at (246.4, 33.4)
- added D10: D, Diode_THT:D_DO-35_SOD27_P7.62mm_Horizontal, F.Cu at (227.4, 55.0)
- added D11: D, Diode_THT:D_DO-35_SOD27_P7.62mm_Horizontal, F.Cu at (227.4, 74.0)
- added D12: D, Diode_THT:D_DO-35_SOD27_P7.62mm_Horizontal, B.Cu at (293.0, 99.7)
- added D13: D, Diode_THT:D_DO-35_SOD27_P7.62mm_Horizontal, F.Cu at (284.6, 38.2)
- added D14: D, Diode_THT:D_DO-35_SOD27_P7.62mm_Horizontal, F.Cu at (284.6, 57.3)
- added D15: D, Diode_THT:D_DO-35_SOD27_P7.62mm_Horizontal, F.Cu at (284.6, 76.4)
- added D16: D, Diode_THT:D_DO-35_SOD27_P7.62mm_Horizontal, F.Cu at (208.4, 40.8)
- added D17: D, Diode_THT:D_DO-35_SOD27_P7.62mm_Horizontal, F.Cu at (208.4, 59.8)
- added D18: D, Diode_THT:D_DO-35_SOD27_P7.62mm_Horizontal, F.Cu at (208.4, 78.8)
- added D19: D, Diode_THT:D_DO-35_SOD27_P7.62mm_Horizontal, F.Cu at (189.4, 40.8)
- added D2: D, Diode_THT:D_DO-35_SOD27_P7.62mm_Horizontal, F.Cu at (246.6, 52.5)
- added D20: D, Diode_THT:D_DO-35_SOD27_P7.62mm_Horizontal, F.Cu at (189.4, 59.8)
- added D21: D, Diode_THT:D_DO-35_SOD27_P7.62mm_Horizontal, F.Cu at (189.4, 78.8)
- added D3: D, Diode_THT:D_DO-35_SOD27_P7.62mm_Horizontal, F.Cu at (246.4, 71.6)
- added D4: D, Diode_THT:D_DO-35_SOD27_P7.62mm_Horizontal, F.Cu at (269.4, 95.4)
- added D5: D, Diode_THT:D_DO-35_SOD27_P7.62mm_Horizontal, F.Cu at (265.6, 36.0)
- added D6: D, Diode_THT:D_DO-35_SOD27_P7.62mm_Horizontal, F.Cu at (265.6, 55.0)
- added D7: D, Diode_THT:D_DO-35_SOD27_P7.62mm_Horizontal, F.Cu at (265.6, 74.0)
- added D8: D, Diode_THT:D_DO-35_SOD27_P7.62mm_Horizontal, B.Cu at (305.9, 87.1)
- added D9: D, Diode_THT:D_DO-35_SOD27_P7.62mm_Horizontal, F.Cu at (227.4, 36.0)
- added H2: MountingHole, TestPoint:TestPoint_Loop_D3.80mm_Drill2.8mm, B.Cu at (300.0, 25.2)
- added H4: MountingHole, TestPoint:TestPoint_Loop_D3.80mm_Drill2.8mm, B.Cu at (229.0, 100.2)
- added H6: MountingHole, TestPoint:TestPoint_Loop_D3.80mm_Drill2.8mm, B.Cu at (192.0, 25.2)
- added H8: MountingHole, TestPoint:TestPoint_Loop_D3.80mm_Drill2.8mm, B.Cu at (316.0, 65.2)
- added R1: R, Resistor_THT:R_Axial_DIN0207_L6.3mm_D2.5mm_P7.62mm_Horizontal, B.Cu at (320.8, 46.2)
- added R2: R, Resistor_THT:R_Axial_DIN0207_L6.3mm_D2.5mm_P7.62mm_Horizontal, B.Cu at (313.2, 52.2)
- added SW1: SW_Push, GateronKS33Solder:Gateron-KS33-Solderable-1U, F.Cu at (256.0, 37.3)
- added SW10: SW_Push, GateronKS33Solder:Gateron-KS33-Solderable-1U, F.Cu at (236.9, 58.7)
- added SW11: SW_Push, GateronKS33Solder:Gateron-KS33-Solderable-1U, F.Cu at (236.9, 77.8)
- added SW12: SW_Push, GateronKS33Solder:Gateron-KS33-Solderable-1U, B.Cu at (282.9, 100.9)
- added SW13: SW_Push, GateronKS33Solder:Gateron-KS33-Solderable-1U, F.Cu at (294.1, 42.0)
- added SW14: SW_Push, GateronKS33Solder:Gateron-KS33-Solderable-1U, F.Cu at (294.1, 61.1)
- added SW15: SW_Push, GateronKS33Solder:Gateron-KS33-Solderable-1U, F.Cu at (294.1, 80.1)
- added SW16: SW_Push, GateronKS33Solder:Gateron-KS33-Solderable-1U, F.Cu at (217.9, 44.4)
- added SW17: SW_Push, GateronKS33Solder:Gateron-KS33-Solderable-1U, F.Cu at (217.9, 63.5)
- added SW18: SW_Push, GateronKS33Solder:Gateron-KS33-Solderable-1U, F.Cu at (217.9, 82.5)
- added SW19: SW_Push, GateronKS33Solder:Gateron-KS33-Solderable-1U, F.Cu at (198.8, 44.5)
- added SW2: SW_Push, GateronKS33Solder:Gateron-KS33-Solderable-1U, F.Cu at (256.0, 56.3)
- added SW20: SW_Push, GateronKS33Solder:Gateron-KS33-Solderable-1U, F.Cu at (198.8, 63.6)
- added SW21: SW_Push, GateronKS33Solder:Gateron-KS33-Solderable-1U, F.Cu at (198.8, 82.6)
- added SW3: SW_Push, GateronKS33Solder:Gateron-KS33-Solderable-1U, F.Cu at (256.0, 75.4)
- added SW4: SW_Push, GateronKS33Solder:Gateron-KS33-Solderable-1U, F.Cu at (259.8, 99.2)
- added SW5: SW_Push, GateronKS33Solder:Gateron-KS33-Solderable-1U, F.Cu at (275.1, 39.7)
- added SW6: SW_Push, GateronKS33Solder:Gateron-KS33-Solderable-1U, F.Cu at (275.1, 58.7)
- added SW7: SW_Push, GateronKS33Solder:Gateron-KS33-Solderable-1U, F.Cu at (275.1, 77.8)
- added SW8: SW_Push, GateronKS33Solder:Gateron-KS33-Solderable-2U, B.Cu at (312.2, 95.2)
- added SW9: SW_Push, GateronKS33Solder:Gateron-KS33-Solderable-1U, F.Cu at (236.9, 39.7)
- added TP1: BAT, TestPoint:TestPoint_Pad_D2.0mm, B.Cu at (331.9, 22.2)
- added TP2: GND, TestPoint:TestPoint_Pad_D2.0mm, B.Cu at (344.0, 22.2)
- added U1: XIAO-nRF52840-SMD, Moddedxiao:modified-XIAO-nRF52840-SMD, F.Cu at (316.0, 30.2)
- moved H1 179.4 mm to (184.0, 25.0), turned to 90 degrees
- moved H3 168.2 mm to (184.0, 46.3), turned to 90 degrees
- moved H5 157.6 mm to (184.0, 67.7), turned to 90 degrees
- moved H7 147.8 mm to (184.0, 89.0), turned to 90 degrees
Routing:
- net Col3: track 185.3 -> 371.1 mm, vias 0 -> 2
- net Row3: track 158.7 -> 328.5 mm
- net Col6: track 165.7 -> 324.0 mm, vias 0 -> 2
- net Row2: track 138.2 -> 288.0 mm
- net Row1: track 127.0 -> 270.8 mm
- net Col5: track 148.1 -> 286.5 mm, vias 0 -> 3
- net Col2: track 145.4 -> 280.1 mm, vias 1 -> 2
- net Col1: track 150.6 -> 278.1 mm, vias 1 -> 2
- net Row4: track 93.7 -> 194.0 mm
- net GND: track 67.8 -> 142.5 mm, vias 0 -> 2
- net Col4: track 69.9 -> 133.0 mm, vias 1 -> 2
- net VBAT: track 30.6 -> 70.1 mm
- net BTPin: track 42.3 -> 74.1 mm, vias 0 -> 1
- net Net-(D8-A): track 16.5 -> 33.1 mm
- net Net-(D6-A): track 7.61 -> 21.8 mm
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Other:
- board size 162 x 94 mm -> 327.9 x 94 mm
- board text added: "left side"

Commit message: firmware framework done
Parts:
- D12, D8, SW12, SW8: moved to F.Cu
- moved D3 1.11 mm to (120.6, 71.4)
- moved SW4 1.11 mm to (107.2, 99.0)
- moved D1 1.11 mm to (120.6, 33.2)
- moved D4 1.11 mm to (97.6, 95.2)
- moved D8 1.11 mm to (61.1, 86.9)
- moved TP1 1.11 mm to (35.1, 22.0)
- moved TP2 1.11 mm to (23.0, 22.0)
- moved U1 1.11 mm to (51.0, 30.0)
- moved H8 1.11 mm to (51.0, 65.0)
- moved R1 1.11 mm to (46.2, 46.0)
- moved SW8 1.11 mm to (54.8, 95.0)
- moved SW3 1.11 mm to (111.0, 75.2)
- moved D2 1.11 mm to (120.4, 52.3)
- moved D5 1.11 mm to (101.4, 35.8)
- moved D6 1.11 mm to (101.4, 54.8)
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Routing:
- net Net-(D8-A): track 33.1 -> 16.5 mm
- net Col2: track 280.1 -> 296.7 mm
- net Col3: track 371.1 -> 360.7 mm
- net Net-(D12-A): track 27.9 -> 21.6 mm
Other:
- board size 327.9 x 94 mm -> 330 x 94 mm

Commit message: just case left
Parts:
- added G***: LOGO, LOGO, F.Cu at (33.0, 60.0)
- added G***: LOGO, LOGO, F.Cu at (337.0, 60.0)

Commit message: quick fix
Parts:
- moved D3 90.2 mm to (137.1, 160.0)
- moved D3 90.2 mm to (263.9, 160.0)
- moved D8 90.2 mm to (77.6, 175.6)
- moved D8 90.2 mm to (323.4, 175.6)
- moved SW17 90.2 mm to (235.4, 151.9)
- moved SW17 90.2 mm to (165.6, 151.9)
- moved SW3 90.2 mm to (127.5, 163.8)
- moved SW3 90.2 mm to (273.5, 163.8)
- moved SW4 90.2 mm to (123.7, 187.6)
- moved SW4 90.2 mm to (277.3, 187.6)
- moved SW5 90.2 mm to (292.6, 128.1)
- moved SW5 90.2 mm to (108.5, 128.1)
- moved SW9 90.2 mm to (254.4, 128.1)
- moved SW9 90.2 mm to (146.6, 128.1)
- moved D1 90.2 mm to (263.9, 121.9)
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Routing:
- net Net-(D8-A): track 16.5 -> 35.0 mm
- net Col2: track 296.7 -> 278.9 mm
