File: PCB V2/Guys-split-keyboard/Guys-split-keyboardV2.kicad_pcb (KiCad board)
At the start: 2 copper layers, 330 x 94 mm, 108 parts, among them SW1 SW_Push, SW10 SW_Push, SW11 SW_Push, SW12 SW_Push, SW13 SW_Push, SW14 SW_Push, SW15 SW_Push, SW16 SW_Push, SW17 SW_Push, SW18 SW_Push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

Commit message: done + quick fix
Parts:
- H2, H4, H6, H8: moved to F.Cu
- turned H2 to 0 degrees
- turned H4 to 0 degrees
- turned H6 to 0 degrees
- turned H8 to 0 degrees
